Commit message: Added kinect to robot model

File: robots/panda.gazebo.xacro (robot description, xacro)
@@ -114,3 +114,55 @@
       </xacro:if>
     </xacro:macro>
+    <!-- GAZEBO OPENNI PLUGIN -->
+    <xacro:macro name="kinect_gazebo" params="name ros_topic">
+      <xacro:property name="M_PI" value="3.1415926"/>
+      <gazebo reference="${name}_link">
+        <sensor type="depth" name="${name}_frame_sensor">
+          <always_on>true</always_on>
+          <update_rate>0</update_rate>
+          <visualize>true</visualize>
+          <camera>
+            <horizontal_fov>${1.0*M_PI/180.0}</horizontal_fov>
+            <image>
+              <format>R8G8B8</format>
+              <width>640</width>
+              <height>480</height>
+            </image>
+            <clip>
+              <near>0.1</near>
+              <far>100</far>
+            </clip>
+            <noise>
+              <type>gaussian</type>
+              <mean>0.0</mean>
+              <stddev>0.005</stddev>
+            </noise>
+          </camera>
+          <plugin name="${name}_controller" filename="libgazebo_ros_openni_kinect.so">
+            <updateRate>0</updateRate>
+            <cameraName>${ros_topic}</cameraName>
+            <frameName>${name}_depth_optical_frame</frameName>
+            <imageTopicName>rgb/image_raw</imageTopicName>
+            <depthImageTopicName>depth/image_raw</depthImageTopicName>
+            <!--pointCloudTopicName>depth_registered/points</pointCloudTopicName-->
+            <pointCloudTopicName>depth/points</pointCloudTopicName>
+            <cameraInfoTopicName>rgb/camera_info</cameraInfoTopicName>
+            <depthImageCameraInfoTopicName>depth_registered/camera_info</depthImageCameraInfoTopicName>
+            <pointCloudCutoff>0.5</pointCloudCutoff>
+            <baseline>0.2</baseline>
+            <hackBaseline>0.0</hackBaseline>
+            <distortionK1>0.0</distortionK1>
+            <distortionK2>0.0</distortionK2>
+            <distortionK3>0.0</distortionK3>
+            <distortionT1>0.0</distortionT1>
+            <distortionT2>0.0</distortionT2>
+            <CxPrime>0.0</CxPrime>
+            <Cx>0.0</Cx>
+            <Cy>0.0</Cy>
+            <focalLength>0.0</focalLength>
+          </plugin>
+        </sensor>
+        <material>Gazebo/Black</material>
+      </gazebo>
+    </xacro:macro>
 </robot>

File: robots/panda_arm_hand.urdf.xacro (robot description, xacro)
@@ -2,10 +2,15 @@
 <robot xmlns:xacro="http://www.ros.org/wiki/xacro" name="panda">
   <xacro:arg name="robot_name" default="panda"/>
-  <xacro:arg name="load_gripper" default="true"/>
+  <xacro:arg name="load_gripper" default="False"/>
   <xacro:arg name="load_gazebo" default="false"/>
+  <xacro:arg name="load_rgbd" default="true"/>
   <xacro:include filename="$(find franka_panda_description)/robots/panda_arm.xacro"/>
   <xacro:if value="$(arg load_gripper)">
     <xacro:include filename="$(find franka_panda_description)/robots/hand.xacro"/>
     <xacro:hand ns="panda" rpy="0 0 ${-pi/4}" connected_to="panda_link8"/>
+  </xacro:if>
+  <xacro:if value="$(arg load_rgbd)">
+    <xacro:include filename="$(find franka_panda_description)/robots/kinect.urdf.xacro"/>
+    <xacro:kinect connected_to="panda_link7" name='kinect'/>
   </xacro:if>
   <xacro:if value="$(arg load_gazebo)">
@@ -15,4 +20,7 @@
     <xacro:panda_gazebo robot_name="$(arg robot_name)" load_gripper="$(arg load_gripper)"/>
     <xacro:panda_transmission robot_name="$(arg robot_name)" load_gripper="$(arg load_gripper)"/>
+    <xacro:if value="$(arg load_rgbd)">
+      <xacro:kinect_gazebo name="kinect" ros_topic="kinect_test" />
+    </xacro:if>
   </xacro:if>
   <xacro:unless value="$(arg load_gazebo)">
